File: phase 5.sch (KiCad schematic (older format))
At the start: 11 parts, among them J4 USB_C_Receptacle_USB2.0, SW1 SW_PUSH, U1 ATMEGA32U2, Y1 Resonator

Commit message: Add files via upload
Parts:
- added R5, R6: 22Ohm, Resistor_SMD:R_0805_2012Metric_Pad1.15x1.40mm_HandSolder, symbol Device:R
- R4: value R -> 10kOhm
Connections:
- net GND: now also R5.2, R6.2
- net row1: now also U1.16 (PB2)
- net at J4.A5 (CC1): now also R5.1
- net at J4.A6 (D+): now also R2.1
- net at J4.A7 (D-), R1.1: now also J4.B7 (D-)
- net at J4.B5 (CC2): now also R6.1
Changed lines of the file:
@@
 	6950 2200 6950 2100
-Wire Wire Line
-	4500 2100 5750 2100
 Wire Wire Line
 	6950 2300 6500 2300
@@
 P 9300 3300
 F 0 "R4" V 9507 3300 50  0000 C CNN
-F 1 "R" V 9416 3300 50  0000 C CNN
+F 1 "10kOhm" V 9416 3300 50  0000 C CNN
 F 2 "Resistor_SMD:R_0805_2012Metric_Pad1.15x1.40mm_HandSolder" V 9230 3300 50  0001 C CNN
 F 3 "~" H 9300 3300 50  0001 C CNN
@@
 	4750 2300 6200 2300
 Wire Wire Line
-	4500 2700 4800 2700
-Wire Wire Line
-	4800 2700 4800 2400
-Wire Wire Line
 	4800 2400 4900 2400
 Wire Wire Line
@@
 Wire Wire Line
 	2300 1650 2300 3000
+Wire Wire Line
+	4500 2800 4800 2800
+Wire Wire Line
+	4500 2700 4750 2700
+Wire Wire Line
+	4750 2700 4750 2600
+Connection ~ 4750 2600
+Wire Wire Line
+	4800 2400 4800 2800
+Wire Wire Line
+	9100 3600 9300 3600
+Wire Wire Line
+	9300 3600 9300 4100
+Wire Wire Line
+	9300 4100 1650 4100
+Wire Wire Line
+	1650 4100 1650 3400
+Connection ~ 1650 3400
+Wire Wire Line
+	4900 2150 4500 2150
+Wire Wire Line
+	4500 2150 4500 2300
+Wire Wire Line
+	4500 2400 4600 2400
+Wire Wire Line
+	4600 2200 4600 2400
+$Comp
+L Device:R R5
+U 1 1 5EFEA4D0
+P 5050 2150
+F 0 "R5" V 5257 2150 50  0000 C CNN
+F 1 "22Ohm" V 5166 2150 50  0000 C CNN
+F 2 "Resistor_SMD:R_0805_2012Metric_Pad1.15x1.40mm_HandSolder" V 4980 2150 50  0001 C CNN
+F 3 "~" H 5050 2150 50  0001 C CNN
+	1    5050 2150
+	0    -1   -1   0
+$EndComp
+Wire Wire Line
+	4500 2100 5750 2100
+$Comp
+L power:GND #PWR0109
+U 1 1 5EFEC5AF
+P 5200 2150
+F 0 "#PWR0109" H 5200 1900 50  0001 C CNN
+F 1 "GND" H 5205 1977 50  0000 C CNN
+F 2 "" H 5200 2150 50  0001 C CNN
+F 3 "" H 5200 2150 50  0001 C CNN
+	1    5200 2150
+	0    -1   -1   0
+$EndComp
+Wire Wire Line
+	4600 2200 5750 2200
+$Comp
+L Device:R R6
+U 1 1 5EFEF7C3
+P 5900 2200
+F 0 "R6" V 6107 2200 50  0000 C CNN
+F 1 "22Ohm" V 6016 2200 50  0000 C CNN
+F 2 "Resistor_SMD:R_0805_2012Metric_Pad1.15x1.40mm_HandSolder" V 5830 2200 50  0001 C CNN
+F 3 "~" H 5900 2200 50  0001 C CNN
+	1    5900 2200
+	0    -1   -1   0
+$EndComp
+$Comp
+L power:GND #PWR0110
+U 1 1 5EFEF7C9
+P 6050 2200
+F 0 "#PWR0110" H 6050 1950 50  0001 C CNN
+F 1 "GND" H 6055 2027 50  0000 C CNN
+F 2 "" H 6050 2200 50  0001 C CNN
+F 3 "" H 6050 2200 50  0001 C CNN
+	1    6050 2200
+	0    -1   -1   0
+$EndComp
 $EndSCHEMATC

Commit message: Add files via upload
Parts:
- removed D_BOTTOM_ENTER1: D, keyboard_parts:D_SOD123_axial, symbol Device:D
- R5, R6: value 22Ohm -> 5.1kohm
Connections:
- net col0: now also U1.8 (PD2/RXD1)
- net row1: now also K_BOTTOM_ENTER1.2
- net at J4.A6 (D+), R2.1: now also J4.B6 (D+)
Changed lines of the file:
@@
 Text GLabel 1400 3400 0    50   Input ~ 0
 row1
-Wire Wire Line
-	1400 3400 1650 3400
-Wire Wire Line
-	1700 3000 1650 3000
-Wire Wire Line
-	1650 3000 1650 3100
 $Comp
 L Connector:USB_C_Receptacle_USB2.0 J4
@@
 	1    0    0    -1
 $EndComp
-Wire Wire Line
-	6950 2200 6950 2100
-Wire Wire Line
-	6950 2300 6500 2300
-Wire Wire Line
-	6100 2500 6950 2500
-Wire Wire Line
-	6950 2600 6400 2600
-Connection ~ 6100 2600
-Wire Wire Line
-	6100 2600 6100 2500
 $Comp
 L power:VCC #PWR0101
@@
 	1    0    0    -1
 $EndComp
-Connection ~ 5750 2100
-Wire Wire Line
-	5750 2100 6950 2100
-Wire Wire Line
-	4050 3600 5800 3600
-Wire Wire Line
-	3900 3700 3900 3600
 $Comp
 L power:GND #PWR0102
@@
 	0    -1   -1   0
 $EndComp
-Wire Wire Line
-	9150 3300 9100 3300
 $Comp
 L power:GND #PWR0103
@@
 	0    -1   -1   0
 $EndComp
-Wire Wire Line
-	3600 3600 3900 3600
-Connection ~ 3600 3600
-Connection ~ 3900 3600
 $Comp
 L Device:R R3
@@
 	1    0    0    -1
 $EndComp
-Wire Wire Line
-	4050 3600 4050 3700
-Wire Wire Line
-	4050 3700 3900 3700
 $Comp
 L power:GND #PWR0104
@@
 	1    0    0    -1
 $EndComp
-Wire Wire Line
-	6200 2950 6200 2900
-Wire Wire Line
-	4500 2600 4750 2600
-Wire Wire Line
-	4750 2600 4750 2300
-Wire Wire Line
-	4750 2300 6200 2300
-Wire Wire Line
-	4800 2400 4900 2400
-Wire Wire Line
-	5200 2400 6950 2400
-Wire Wire Line
-	6100 2600 5800 2600
-Wire Wire Line
-	5800 2600 5800 3600
-Connection ~ 6950 2100
 $Comp
 L keyboard_parts:ATMEGA32U2 U1
@@
 	-1   0    0    -1
 $EndComp
-Wire Wire Line
-	6800 2900 6850 2900
-Wire Wire Line
-	6850 2700 6850 2900
-Connection ~ 6850 2900
-Wire Wire Line
-	6850 2900 6950 2900
-Wire Wire Line
-	6400 2700 6550 2700
 $Comp
 L power:VCC #PWR0105
@@
 	0    -1   -1   0
 $EndComp
-Wire Wire Line
-	9200 2300 9100 2300
 $Comp
 L Device:Resonator Y1
@@
 	0    -1   -1   0
 $EndComp
-Wire Wire Line
-	10050 1950 9100 1950
-Wire Wire Line
-	9100 1950 9100 2100
-Wire Wire Line
-	10050 2250 9550 2250
-Wire Wire Line
-	9550 2250 9550 2200
-Wire Wire Line
-	9550 2200 9100 2200
 $Comp
 L Device:C C1
@@
 $EndComp
 $Comp
-L Device:D D_BOTTOM_ENTER1
-U 1 1 5EFD96A7
-P 1650 3250
-F 0 "D_BOTTOM_ENTER1" V 1696 3171 50  0000 R CNN
-F 1 "D" V 1595 3171 50  0000 R CNN
-F 2 "keyboard_parts:D_SOD123_axial" H 1650 3250 50  0001 C CNN
-F 3 "~" H 1650 3250 50  0001 C CNN
-	1    1650 3250
-	0    -1   -1   0
-$EndComp
-Wire Wire Line
-	2300 1650 2300 3000
-Wire Wire Line
-	4500 2800 4800 2800
-Wire Wire Line
-	4500 2700 4750 2700
-Wire Wire Line
-	4750 2700 4750 2600
-Connection ~ 4750 2600
-Wire Wire Line
-	4800 2400 4800 2800
-Wire Wire Line
-	9100 3600 9300 3600
-Wire Wire Line
-	9300 3600 9300 4100
-Wire Wire Line
-	9300 4100 1650 4100
-Wire Wire Line
-	1650 4100 1650 3400
-Connection ~ 1650 3400
-Wire Wire Line
-	4900 2150 4500 2150
-Wire Wire Line
-	4500 2150 4500 2300
-Wire Wire Line
-	4500 2400 4600 2400
-Wire Wire Line
-	4600 2200 4600 2400
-$Comp
 L Device:R R5
 U 1 1 5EFEA4D0
 P 5050 2150
 F 0 "R5" V 5257 2150 50  0000 C CNN
-F 1 "22Ohm" V 5166 2150 50  0000 C CNN
+F 1 "5.1kohm" V 5166 2150 50  0000 C CNN
 F 2 "Resistor_SMD:R_0805_2012Metric_Pad1.15x1.40mm_HandSolder" V 4980 2150 50  0001 C CNN
 F 3 "~" H 5050 2150 50  0001 C CNN
@@
 	0    -1   -1   0
 $EndComp
-Wire Wire Line
-	4500 2100 5750 2100
 $Comp
 L power:GND #PWR0109
@@
 	0    -1   -1   0
 $EndComp
-Wire Wire Line
-	4600 2200 5750 2200
 $Comp
 L Device:R R6
@@
 P 5900 2200
 F 0 "R6" V 6107 2200 50  0000 C CNN
-F 1 "22Ohm" V 6016 2200 50  0000 C CNN
+F 1 "5.1kohm" V 6016 2200 50  0000 C CNN
 F 2 "Resistor_SMD:R_0805_2012Metric_Pad1.15x1.40mm_HandSolder" V 5830 2200 50  0001 C CNN
 F 3 "~" H 5900 2200 50  0001 C CNN
@@
 	0    -1   -1   0
 $EndComp
+Wire Wire Line
+	1400 3400 1650 3400
+Wire Wire Line
+	1700 3000 1650 3000
+Wire Wire Line
+	6950 2200 6950 2100
+Wire Wire Line
+	6950 2300 6500 2300
+Wire Wire Line
+	6100 2500 6950 2500
+Wire Wire Line
+	6950 2600 6400 2600
+Connection ~ 6100 2600
+Wire Wire Line
+	6100 2600 6100 2500
+Connection ~ 5750 2100
+Wire Wire Line
+	5750 2100 6950 2100
+Wire Wire Line
+	4050 3600 5800 3600
+Wire Wire Line
+	3900 3700 3900 3600
+Wire Wire Line
+	9150 3300 9100 3300
+Wire Wire Line
+	3600 3600 3900 3600
+Connection ~ 3600 3600
+Connection ~ 3900 3600
+Wire Wire Line
+	4050 3600 4050 3700
+Wire Wire Line
+	4050 3700 3900 3700
+Wire Wire Line
+	6200 2950 6200 2900
+Wire Wire Line
+	4500 2600 4750 2600
+Wire Wire Line
+	4750 2600 4750 2300
+Wire Wire Line
+	4750 2300 6200 2300
+Wire Wire Line
+	4800 2400 4900 2400
+Wire Wire Line
+	5200 2400 6950 2400
+Wire Wire Line
+	6100 2600 5800 2600
+Wire Wire Line
+	5800 2600 5800 3600
+Connection ~ 6950 2100
+Wire Wire Line
+	6800 2900 6850 2900
+Wire Wire Line
+	6850 2700 6850 2900
+Connection ~ 6850 2900
+Wire Wire Line
+	6850 2900 6950 2900
+Wire Wire Line
+	6400 2700 6550 2700
+Wire Wire Line
+	9200 2300 9100 2300
+Wire Wire Line
+	10050 1950 9100 1950
+Wire Wire Line
+	9100 1950 9100 2100
+Wire Wire Line
+	10050 2250 9550 2250
+Wire Wire Line
+	9550 2250 9550 2200
+Wire Wire Line
+	9550 2200 9100 2200
+Wire Wire Line
+	4500 2800 4800 2800
+Wire Wire Line
+	4500 2700 4750 2700
+Wire Wire Line
+	4750 2700 4750 2600
+Connection ~ 4750 2600
+Wire Wire Line
+	4800 2400 4800 2800
+Wire Wire Line
+	4900 2150 4500 2150
+Wire Wire Line
+	4500 2150 4500 2300
+Wire Wire Line
+	4500 2400 4600 2400
+Wire Wire Line
+	4600 2200 4600 2400
+Wire Wire Line
+	4500 2100 5750 2100
+Wire Wire Line
+	4600 2200 5750 2200
+Wire Wire Line
+	4500 2900 4800 2900
+Wire Wire Line
+	4800 2900 4800 2800
+Connection ~ 4800 2800
+Wire Wire Line
+	1650 3000 1650 3400
+Text GLabel 9100 2800 2    50   Input ~ 0
+col0
+Wire Wire Line
+	2300 1650 2300 3000
+Text GLabel 9100 3600 2    50   Input ~ 0
+row1
 $EndSCHEMATC
