File: phase 5.kicad_pcb (KiCad board)
At the start: 2 copper layers, 48.9 x 44.1 mm, 13 parts, among them J4 USB_C_Receptacle_USB2.0, SW1 SW_PUSH, U1 ATMEGA32U2, Y1 Resonator

Commit message: Add files via upload
Parts:
- removed D_BOTTOM_ENTER: D, keyboard_parts:D_SOD123_axial
- added D_BOTTOM_ENTER1: D, keyboard_parts:D_SOD123_axial, F.Cu at (20.0, 49.1)
- added R5: 22Ohm, Resistor_SMD:R_0805_2012Metric_Pad1.15x1.40mm_HandSolder, F.Cu at (54.0, 24.4)
- added R6: 22Ohm, Resistor_SMD:R_0805_2012Metric_Pad1.15x1.40mm_HandSolder, F.Cu at (54.0, 19.7)
- R4: value R -> 10kOhm
- moved R3 33.3 mm to (32.0, 28.9)
- moved C1 24.2 mm to (39.0, 41.3)
- moved Y1 20.6 mm to (60.5, 32.2)
- moved R4 17.5 mm to (45.1, 32.9)
- moved R1 16.8 mm to (38.5, 35.0)
- moved R2 14.5 mm to (45.2, 37.5)
Connections:
- net col0 renamed Net-(U1-Pad21)
- J4 pad B7: Net-(J4-PadB7) -> Net-(J4-PadA7)
- R2 pad 1: Net-(J4-PadB7) -> Net-(J4-PadA6)
- U1 pad 16: Net-(U1-Pad16) -> row1
Routing:
- net /col0: track 1.63 -> 0.00 mm

Commit message: Add files via upload
Parts:
- removed D_BOTTOM_ENTER1: D, keyboard_parts:D_SOD123_axial
- HOLE_M2.6 (x2): value VAL** -> M2 Whole
- R5, R6: value 22Ohm -> 5.1kohm
- moved Y1 28.1 mm to (32.4, 33.7)
- moved R3 22.1 mm to (52.9, 36.2)
- moved R2 11.7 mm to (39.9, 27.0)
- moved R1 9.53 mm to (43.9, 27.1)
- moved R4 7.71 mm to (52.8, 32.8)
- moved U1 3.57 mm to (41.1, 34.6)
- moved C1 2.77 mm to (41.7, 41.2)
- moved R5 2.51 mm to (56.5, 24.6)
- moved R6 2.43 mm to (56.4, 19.8)
Connections:
- J4 pad B6: Net-(J4-PadB6) -> Net-(J4-PadA6)
- K_BOTTOM_ENTER pad 1: Net-(K_BOTTOM_ENTER-Pad1) -> col0
- U1 pad 8: Net-(U1-Pad8) -> col0
Routing:
- net Net-(D_BOTTOM_ENTER-Pad2): track 25.1 -> 0.00 mm
Other:
- board text added: "."

Commit message: Add files via upload
Parts:
- removed the HOLE_M2.6 at (20.5, 57.9)
- removed the HOLE_M2.6 at (62.7, 19.8)
- added HOLE_M2.6: VAL**, keyboard_parts:HOLE_M2.6, F.Cu at (62.5, 19.9)
- added HOLE_M2.6: VAL**, keyboard_parts:HOLE_M2.6, F.Cu at (20.3, 58.5)
Connections:
- K_BOTTOM_ENTER pad 1: col0 -> (no net)
- K_BOTTOM_ENTER pad 2: Net-(D_BOTTOM_ENTER-Pad2) -> (no net)
- U1 pad 16: row1 -> (no net)
- U1 pad 8: col0 -> (no net)
Routing:
- net Net-(R3-Pad2): track 0.00 -> 49.1 mm
- net Net-(R2-Pad2): track 0.00 -> 33.5 mm
- net (no net): track 0.00 -> 29.9 mm, vias 1 -> 2
- net Net-(R1-Pad2): track 0.00 -> 13.6 mm, vias 0 -> 2
- net Net-(J4-PadB5): track 0.00 -> 13.5 mm
- net Net-(J4-PadA6): track 0.00 -> 12.6 mm
- net Net-(R4-Pad1): track 0.00 -> 12.6 mm, vias 0 -> 2
- net Net-(J4-PadA5): track 0.00 -> 10.9 mm
- net Net-(U1-Pad2): track 0.00 -> 10.3 mm
- net Net-(J4-PadA7): track 0.00 -> 5.51 mm
- net Net-(U1-Pad1): track 0.00 -> 4.69 mm
- net GND: track 0.00 -> 2.92 mm, vias 0 -> 3
- net Net-(C1-Pad2): track 0.00 -> 2.64 mm

Commit message: Add files via upload
Parts:
- removed HOLE_M2.6 (x2): VAL**, keyboard_parts:HOLE_M2.6
- added ?: MountingHole_2.1mm, MountingHole:MountingHole_2.1mm, F.Cu at (62.5, 58.1)
- added ?: MountingHole_2.1mm, MountingHole:MountingHole_2.1mm, F.Cu at (62.5, 20.1)
- added ?: MountingHole_2.1mm, MountingHole:MountingHole_2.1mm, F.Cu at (20.3, 58.1)
- added REF**: MountingHole_2.1mm, MountingHole:MountingHole_2.1mm, F.Cu at (20.3, 39.5)
